Commit message: 1

File: SmarticleLowProfileThicker.urdf (robot description, URDF)
Before this commit: robot SmarticleLowProfile, 3 links, 2 joints
Links:
- link arm1: geometry collision box size=0.005 0.05 0.005; visual box size=0.005 0.05 0.005
- link arm2: geometry collision box size=0.005 0.05 0.005; visual box size=0.005 0.05 0.005
- link base_link: geometry collision box size=0.015 0.05 0.005; visual box size=0.015 0.05 0.005
Joints:
- joint j_1: origin xyz=0 0.0225 0.00011 rpy=0 0 0 -> xyz=0 0.0225 0.0001 rpy=0 0 0
- joint j_2: origin xyz=0 -0.0225 0.0011 rpy=0 0 0 -> xyz=0 -0.0225 0.001 rpy=0 0 0
